File: display/display.kicad_pcb (KiCad board)
At the start: 4 copper layers, 116.7 x 41.4 mm, 40 parts, among them J1 Conn_01x08_Pin, J2 Conn_01x08_Pin, Q1 BSS84, Q2 BSS84, Q3 BSS84, Q4 BSS84, Q5 BSS84, Q6 BSS84, Q7 BSS84, Q8 BSS84, SW1 SW_Push, SW2 SW_Push, SW3 SW_Push, SW4 SW_Push, SW5 SW_Push, SW6 SW_Push, U1 STP16CPC26M, U2 STP16CPC26M, U3 STP16CPC26M

Commit message: MUX prepoje na druhej polke 16 seg displejov
Routing:
- net Net-(DS1-CA_1): track 0.00 -> 9.76 mm
- net Net-(DS2-CA_1): track 0.00 -> 8.96 mm
- net Net-(DS1-CA_2): track 0.00 -> 8.44 mm
- net Net-(J1-Pin_7): track 115.1 -> 116.6 mm
Changed lines of the file:
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@@
 	)
 	(segment
+		(start 173.7057 73.2936)
+		(end 173.7057 71.8484)
+		(width 0.4)
+		(layer "F.Cu")
+		(net "Net-(J1-Pin_7)")
+	)
+	(segment
 		(start 90.020761 68.184349)
 		(end 90.12031 68.0848)
@@
 	)
 	(segment
-		(start 173.7057 73.2936)
+		(start 173.8181 74.9808)
 		(end 173.8181 73.406)
 		(width 0.4)
@@
 	)
 	(segment
-		(start 173.7057 71.8484)
+		(start 173.8181 73.406)
 		(end 173.7057 73.2936)
 		(width 0.4)
@@
 	)
 	(via
-		(at 173.8181 73.406)
+		(at 173.8181 74.9808)
 		(size 0.6)
 		(drill 0.3)
@@
 	)
 	(segment
-		(start 173.8181 73.406)
-		(end 173.8181 83.3232)
-		(width 0.4)
-		(layer "In1.Cu")
-		(net "Net-(J1-Pin_7)")
-	)
-	(segment
 		(start 138.4172 69.4182)
 		(end 138.8998 69.9008)
@@
 	)
 	(segment
+		(start 173.8181 74.9808)
+		(end 173.8181 83.3232)
+		(width 0.4)
+		(layer "In1.Cu")
+		(net "Net-(J1-Pin_7)")
+	)
+	(segment
 		(start 117.330579 75.3842)
 		(end 118.055979 76.1096)
@@
 	)
 	(segment
-		(start 134.239 75.7936)
-		(end 134.239 76.045271)
+		(start 173.8181 83.3232)
+		(end 175.0161 84.5212)
 		(width 0.4)
 		(layer "In1.Cu")
@@
 	)
 	(segment
-		(start 173.8181 83.3232)
-		(end 175.0161 84.5212)
+		(start 134.239 75.7936)
+		(end 134.239 76.045271)
 		(width 0.4)
 		(layer "In1.Cu")
@@
 	)
 	(segment
-		(start 159.5628 72.898)
-		(end 173.3101 72.898)
+		(start 173.3101 72.898)
+		(end 159.5628 72.898)
 		(width 0.4)
 		(layer "In2.Cu")
@@
 	)
 	(segment
-		(start 156.5656 69.9008)
-		(end 159.5628 72.898)
+		(start 159.5628 72.898)
+		(end 156.5656 69.9008)
 		(width 0.4)
 		(layer "In2.Cu")
@@
 	)
 	(segment
-		(start 173.3101 72.898)
+		(start 173.8181 74.9808)
 		(end 173.8181 73.406)
 		(width 0.4)
@@
 	)
 	(segment
-		(start 138.8998 69.9008)
-		(end 156.5656 69.9008)
+		(start 173.8181 73.406)
+		(end 173.3101 72.898)
+		(width 0.4)
+		(layer "In2.Cu")
+		(net "Net-(J1-Pin_7)")
+	)
+	(segment
+		(start 156.5656 69.9008)
+		(end 138.8998 69.9008)
 		(width 0.4)
 		(layer "In2.Cu")
@@
 	)
 	(segment
+		(start 154.5208 75.0171)
+		(end 154.5208 73.328629)
+		(width 0.4)
+		(layer "B.Cu")
+		(net "Net-(DS2-CA_1)")
+	)
+	(segment
+		(start 154.5208 73.328629)
+		(end 150.1147 68.922529)
+		(width 0.4)
+		(layer "B.Cu")
+		(net "Net-(DS2-CA_1)")
+	)
+	(segment
+		(start 150.1147 68.922529)
+		(end 150.1147 68.0788)
+		(width 0.4)
+		(layer "B.Cu")
+		(net "Net-(DS2-CA_1)")
+	)
+	(segment
+		(start 154.3797 75.1582)
+		(end 154.5208 75.0171)
+		(width 0.4)
+		(layer "B.Cu")
+		(net "Net-(DS2-CA_1)")
+	)
+	(segment
 		(start 138.0998 68.0937)
 		(end 138.1147 68.0788)
@@
 	)
 	(segment
+		(start 158.5109 69.5347)
+		(end 158.5109 68.0542)
+		(width 0.4)
+		(layer "B.Cu")
+		(net "Net-(DS1-CA_2)")
+	)
+	(segment
+		(start 158.0371 75.053692)
+		(end 159.8871 73.203692)
+		(width 0.4)
+		(layer "B.Cu")
+		(net "Net-(DS1-CA_2)")
+	)
+	(segment
+		(start 159.8871 73.203692)
+		(end 159.8871 70.9109)
+		(width 0.4)
+		(layer "B.Cu")
+		(net "Net-(DS1-CA_2)")
+	)
+	(segment
+		(start 159.8871 70.9109)
+		(end 158.5109 69.5347)
+		(width 0.4)
+		(layer "B.Cu")
+		(net "Net-(DS1-CA_2)")
+	)
+	(segment
+		(start 158.0371 75.1582)
+		(end 158.0371 75.053692)
+		(width 0.4)
+		(layer "B.Cu")
+		(net "Net-(DS1-CA_2)")
+	)
+	(segment
+		(start 170.5109 70.2063)
+		(end 170.8404 70.5358)
+		(width 0.4)
+		(layer "B.Cu")
+		(net "Net-(DS1-CA_1)")
+	)
+	(segment
+		(start 174.0408 73.8139)
+		(end 175.2327 75.0058)
+		(width 0.4)
+		(layer "B.Cu")
+		(net "Net-(DS1-CA_1)")
+	)
+	(segment
+		(start 174.0408 72.2884)
+		(end 174.0408 73.8139)
+		(width 0.4)
+		(layer "B.Cu")
+		(net "Net-(DS1-CA_1)")
+	)
+	(segment
+		(start 170.8404 70.5358)
+		(end 172.2882 70.5358)
+		(width 0.4)
+		(layer "B.Cu")
+		(net "Net-(DS1-CA_1)")
+	)
+	(segment
+		(start 170.5109 68.0542)
+		(end 170.5109 70.2063)
+		(width 0.4)
+		(layer "B.Cu")
+		(net "Net-(DS1-CA_1)")
+	)
+	(segment
+		(start 172.2882 70.5358)
+		(end 174.0408 72.2884)
+		(width 0.4)
+		(layer "B.Cu")
+		(net "Net-(DS1-CA_1)")
+	)
+	(segment

Commit message: Jedna cesta a SW priešinok.
Routing:
- net Net-(DS1-CATODE_K): track 7.20 -> 57.3 mm, vias 1 -> 2
Changed lines of the file:
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@@
+	)
+	(segment
+		(start 157.4038 70.776029)
+		(end 157.4038 57.6072)
+		(width 0.4)
+		(layer "F.Cu")
+		(net "Net-(DS1-CATODE_K)")
+	)
+	(segment
+		(start 157.4038 57.6072)
+		(end 156.2354 57.6072)
+		(width 0.4)
+		(layer "F.Cu")
+		(net "Net-(DS1-CATODE_K)")
+	)
+	(segment
+		(start 154.1147 56.7565)
+		(end 154.1147 55.3788)
+		(width 0.4)
+		(layer "F.Cu")
+		(net "Net-(DS1-CATODE_K)")
+	)
+	(segment
+		(start 153.840682 74.671489)
+		(end 156.3498 72.162371)
+		(width 0.4)
+		(layer "F.Cu")
+		(net "Net-(DS1-CATODE_K)")
+	)
+	(segment
+		(start 154.9654 57.6072)
+		(end 154.1147 56.7565)
+		(width 0.4)
+		(layer "F.Cu")
+		(net "Net-(DS1-CATODE_K)")
+	)
+	(segment
+		(start 156.3498 71.830029)
+		(end 157.4038 70.776029)
+		(width 0.4)
+		(layer "F.Cu")
+		(net "Net-(DS1-CATODE_K)")
+	)
+	(segment
+		(start 156.3498 72.162371)
+		(end 156.3498 71.830029)
+		(width 0.4)
+		(layer "F.Cu")
+		(net "Net-(DS1-CATODE_K)")
+	)
+	(segment
+		(start 153.33335 74.671489)
+		(end 153.840682 74.671489)
+		(width 0.4)
+		(layer "F.Cu")
+		(net "Net-(DS1-CATODE_K)")
+	)
+	(segment
+		(start 156.2354 57.6072)
+		(end 174.0408 57.6072)
+		(width 0.4)
+		(layer "F.Cu")
+		(net "Net-(DS1-CATODE_K)")
+	)
+	(segment
+		(start 174.0408 57.6072)
+		(end 174.5109 57.1371)
+		(width 0.4)
+		(layer "F.Cu")
+		(net "Net-(DS1-CATODE_K)")
+	)
+	(segment
+		(start 156.2354 57.6072)
+		(end 154.9654 57.6072)
+		(width 0.4)
+		(layer "F.Cu")
+		(net "Net-(DS1-CATODE_K)")
+	)
+	(segment
+		(start 174.5109 57.1371)
+		(end 174.5109 55.3542)
+		(width 0.4)
+		(layer "F.Cu")
+		(net "Net-(DS1-CATODE_K)")
 	)
 	(segment
@@
 		(net "Net-(DS1-CATODE_K)")
 	)
+	(via
+		(at 153.33335 74.671489)
+		(size 0.6)
+		(drill 0.3)
+		(layers "F.Cu" "B.Cu")
+		(net "Net-(DS1-CATODE_K)")
+	)
+	(segment
+		(start 153.33335 74.671489)
+		(end 153.553371 74.89151)
+		(width 0.4)
+		(layer "In2.Cu")
+		(net "Net-(DS1-CATODE_K)")
+	)
+	(segment
+		(start 155.787298 77.138527)
+		(end 155.787298 79.4258)
+		(width 0.4)
+		(layer "In2.Cu")
+		(net "Net-(DS1-CATODE_K)")
+	)
+	(segment
+		(start 153.553371 74.9046)
+		(end 155.787298 77.138527)
+		(width 0.4)
+		(layer "In2.Cu")
+		(net "Net-(DS1-CATODE_K)")
+	)
+	(segment
+		(start 153.553371 74.89151)
+		(end 153.553371 74.9046)
+		(width 0.4)
+		(layer "In2.Cu")
+		(net "Net-(DS1-CATODE_K)")
+	)

Commit message: nejake cesty
Routing:
- net Net-(DS1-CATODE_U): track 0.00 -> 65.2 mm, vias 0 -> 1
- net Net-(DS1-CATODE_R): track 0.00 -> 47.1 mm, vias 0 -> 3
- net Net-(DS1-CATODE_T): track 0.00 -> 41.1 mm, vias 0 -> 3
- net Net-(DS1-CATODE_S): track 0.00 -> 41.1 mm, vias 0 -> 3
- net Net-(U1-SDO): track 44.8 -> 48.2 mm
- net MUX1: track 35.3 -> 34.4 mm
- net Net-(J1-Pin_5): track 105.5 -> 106.2 mm
- net Net-(J1-Pin_6): track 69.8 -> 70.3 mm

Commit message: nejake cesty
Signed-off-by: RomanGalbi06 <romangalbavy06@gmail.com>
Routing:
- net Net-(DS1-CATODE_N): track 0.00 -> 93.4 mm, vias 0 -> 2
- net Net-(DS1-CATODE_P): track 0.00 -> 92.2 mm, vias 0 -> 1
- net Net-(DS1-CATODE_B): track 0.00 -> 82.3 mm, vias 0 -> 2
- net Net-(DS1-CATODE_M): track 0.00 -> 80.8 mm, vias 0 -> 2
- net Net-(DS1-CATODE_A): track 0.00 -> 76.4 mm
- net Net-(J1-Pin_7): track 116.6 -> 119.1 mm
- net MUX2: track 45.1 -> 47.4 mm
- net MUX1: track 34.4 -> 35.3 mm
- net Net-(U1-SDO): track 48.2 -> 48.8 mm

Commit message: Asi komplet idem pustiť DRC
Signed-off-by: RomanGalbi06 <romangalbavy06@gmail.com>
Routing:
- net Net-(DS1-CATODE_H): track 0.00 -> 74.9 mm, vias 0 -> 3
- net Net-(DS1-CATODE_C): track 0.00 -> 59.8 mm, vias 0 -> 1
- net Net-(DS1-CATODE_F): track 0.00 -> 54.8 mm, vias 0 -> 1
- net Net-(J1-Pin_6): track 70.3 -> 116.6 mm, vias 3 -> 5
- net Net-(DS1-CATODE_E): track 0.00 -> 31.5 mm, vias 0 -> 1
- net Net-(DS1-CATODE_D): track 0.00 -> 30.3 mm, vias 0 -> 1
- net Net-(DS1-CATODE_G): track 0.00 -> 27.9 mm, vias 0 -> 1
- net Net-(R3-Pad2): track 33.1 -> 28.2 mm
- net Net-(U1-SDO): track 48.8 -> 48.1 mm
- net Net-(R4-Pad2): track 48.6 -> 49.3 mm
- net Net-(DS1-CATODE_T): track 41.1 -> 41.7 mm

Commit message: Via Stitching
Signed-off-by: RomanGalbi06 <romangalbavy06@gmail.com>
Routing:
- net GND: vias 6 -> 142

Commit message: no asi final už len poriešiť drc upozernenia
Routing:
- net Net-(DS1-CATODE_P): track 91.8 -> 88.7 mm
- net Net-(DS1-CATODE_U): track 65.6 -> 67.8 mm
- net Net-(DS1-CATODE_C): track 59.8 -> 57.8 mm
- net Net-(DS1-CATODE_N): track 93.4 -> 91.9 mm
- net Net-(DS1-CATODE_M): track 80.8 -> 79.2 mm
- net Net-(DS2-CA_2): track 10.0 -> 11.1 mm
- net Net-(DS1-CATODE_H): track 74.9 -> 74.2 mm
- net GND: vias 142 -> 211

Commit message: no zšiel by sa na PCB ceck či to tak može byť
Routing:
- net Net-(R2-Pad2): track 30.4 -> 25.9 mm
- net Net-(DS3-CATODE_A): track 57.0 -> 54.7 mm
- net Net-(J2-Pin_8): track 141.2 -> 139.0 mm
- net Net-(J1-Pin_6): track 116.6 -> 115.0 mm
- net Net-(DS3-CATODE_K): track 108.2 -> 106.9 mm
- net Net-(DS1-CATODE_F): track 54.8 -> 53.8 mm
- net Net-(DS3-CATODE_B): track 67.8 -> 66.8 mm
- net +5V: track 265.2 -> 264.6 mm
- net Net-(J1-Pin_7): track 119.1 -> 118.5 mm
- net Net-(DS1-CATODE_N): track 91.9 -> 91.3 mm
- net GND: vias 211 -> 242
